File: POWER_LINES.kicad_sch (KiCad schematic)
At the start: 48 parts, among them J6 1730405, J8 1717020, J9 1717020, K3 G2R-1A-E DC5, K4 G2R-1A-E DC5, K5 G2R-1A-E DC5, K6 G2R-1A-E DC5, Q3 AO3400A, Q4 AO3400A, SW2 SW_DPST

Commit message: Footprint assignment
Parts:
- removed SW2: SW_DPST, Button_Switch_THT:SW_NKK_GW12LJP, symbol Switch:SW_DPST
- added J11, J12: 1717020, SmartSupplyLib:CONN_1717020_PXC, symbol SmartSupplyLib:1717020
- C39, C40, C41, C42, C43, C44, C45, C46: footprint (none) -> Capacitor_SMD:C_0805_2012Metric
- H5: footprint 00318201G -> SmartSupplyLib:fuse holder
- J6: footprint CONN_1730405_PXC -> SmartSupplyLib:CONN_1730405_PXC
- J8, J9: footprint CONN_1717020_PXC -> SmartSupplyLib:CONN_1717020_PXC
- K3, K4, K5, K6: footprint RELAY_G2R-1A-E AC12_OMR -> SmartSupplyLib:RELAY_G2R-1A-E AC12_OMR
- R26, R27: footprint Package_DIP:DIP-8_W7.62mm -> Resistor_THT:R_Axial_DIN0414_L11.9mm_D4.5mm_P20.32mm_Horizontal
- R28, R29, R30, R31, R32, R33, R34, R36, R37, R38, R39, R40, R41, R42, R43, R50, R51, R52, R53: footprint Package_DIP:DIP-8_W7.62mm -> Resistor_SMD:R_0805_2012Metric
Connections:
- net CH1_N: now also J12.2
- net L: now also J11.1
- net N: now also J11.2
- net at H5.1: now also J12.1
Other:
- note added: "DPST SWITCH"
- moved on the sheet: H5, J8, J9

Commit message: MOV
Parts:
- added RV1: MOV-14D241K, SmartSupplyLib:MOV14D241K, symbol SmartSupplyLib:MOV-14D241K
Connections:
- net L: now also RV1.2
- net N: now also RV1.1
Other:
- moved on the sheet: J11

Commit message: MOV2
Connections:
- net CH1_L: now also RV1.2
- net CH1_N: now also RV1.1
- net L: no longer RV1.2
- net N: no longer RV1.1
Other:
- moved on the sheet: H5, J8, J9
