File: mcu.kicad_sch (KiCad schematic)
At the start: 31 parts, among them IC4 MIC39100-3.3WS, J1 USB_C_Receptacle_USB2.0_16P, J10 DM3AT-SF-PEJM5, SW1 SW_Push, U1 ESP32-S3-MINI-1U, U4 HLK-10M05

Commit message: 3v3 diodes
Parts:
- added D14: TPD1E10B06DPYR, SmartSupplyLib:TPD1E10B06DPYR, symbol SmartSupplyLib:TPD1E10B06DPYR
Connections:
- net +3.3V: now also D14.1
- net GND: now also D14.2
Changed lines of the file:
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@@
 	(rectangle
 		(start 116.84 90.17)
-		(end 166.37 138.43)
+		(end 204.724 138.43)
 		(stroke
 			(width 0)
@@
 	)
 	(junction
+		(at 158.75 123.19)
+		(diameter 0)
+		(color 0 0 0 0)
+	)
+	(junction
 		(at 86.36 139.7)
 		(diameter 0)
@@
 	(junction
 		(at 58.42 100.33)
+		(diameter 0)
+		(color 0 0 0 0)
+	)
+	(junction
+		(at 158.75 101.6)
 		(diameter 0)
 		(color 0 0 0 0)
@@
 	(wire
 		(pts
+			(xy 173.99 121.92) (xy 173.99 123.19)
+		)
+		(stroke
+			(width 0)
+			(type default)
+		)
+	)
+	(wire
+		(pts
 			(xy 45.72 82.55) (xy 45.72 81.28)
 		)
@@
 	(wire
 		(pts
+			(xy 158.75 101.6) (xy 173.99 101.6)
+		)
+		(stroke
+			(width 0)
+			(type default)
+		)
+	)
+	(wire
+		(pts
 			(xy 97.79 58.42) (xy 97.79 60.96)
 		)
@@
 		(pts
 			(xy 157.48 101.6) (xy 158.75 101.6)
+		)
+		(stroke
+			(width 0)
+			(type default)
+		)
+	)
+	(wire
+		(pts
+			(xy 158.75 123.19) (xy 173.99 123.19)
 		)
 		(stroke
@@
 					(unit 1)
 				)
+			)
+		)
+	)
+	(symbol
+		(lib_id "SmartSupplyLib:TPD1E10B06DPYR")
+		(at 173.99 101.6 270)
+		(unit 1)
+		(body_style 1)
+		(exclude_from_sim no)
+		(in_bom yes)
+		(on_board yes)
+		(in_pos_files yes)
+		(dnp no)
+		(fields_autoplaced yes)
+		(property "Reference" "D14"
+			(at 177.8 110.4899 90)
+			(show_name no)
+			(do_not_autoplace no)
+			(effects
+				(font
+					(size 1.27 1.27)
+				)
+				(justify left)
+			)
+		)
+		(property "Value" "TPD1E10B06DPYR"
+			(at 177.8 113.0299 90)
+			(show_name no)
+			(do_not_autoplace no)
+			(effects
+				(font
+					(size 1.27 1.27)
+				)
+				(justify left)
+			)
+		)
+		(property "Footprint" "SmartSupplyLib:TPD1E10B06DPYR"
+			(at 80.34 114.3 0)
+			(hide yes)
+			(show_name no)
+			(do_not_autoplace no)
+			(effects
+				(font
+					(size 1.27 1.27)
+				)
+				(justify left bottom)
+			)
+		)
+		(property "Datasheet" ""
+			(at -19.66 114.3 0)
+			(hide yes)
+			(show_name no)
+			(do_not_autoplace no)
+			(effects
+				(font
+					(size 1.27 1.27)
+				)
+				(justify left bottom)
+			)
+		)
+		(property "Description" "ESD Suppressors / TVS Diodes Sgl Channel ESD TPD1E10B06 Single-Channel ESD Protection Diode in 0402 Package"
+			(at 173.99 101.6 0)
+			(hide yes)
+			(show_name no)
+			(do_not_autoplace no)
+			(effects
+				(font
+					(size 1.27 1.27)
+				)
+			)
+		)
+		(property "Height" "0.45"
+			(at -219.66 114.3 0)
+			(hide yes)
+			(show_name no)
+			(do_not_autoplace no)
+			(effects
+				(font
+					(size 1.27 1.27)
+				)
+				(justify left bottom)
+			)
+		)
+		(property "Mouser Part Number" "595-TPD1E10B06DPYR"
+			(at -319.66 114.3 0)
+			(hide yes)
+			(show_name no)
+			(do_not_autoplace no)
+			(effects
+				(font
+					(size 1.27 1.27)
+				)
+				(justify left bottom)
+			)
+		)
+		(property "Mouser Price/Stock" "https://www.mouser.co.uk/ProductDetail/Texas-Instruments/TPD1E10B06DPYR?qs=UFc95S4Z4CaJYpQ4xqTc0g%3D%3D"
+			(at -419.66 114.3 0)
+			(hide yes)
+			(show_name no)
+			(do_not_autoplace no)
+			(effects
+				(font
+					(size 1.27 1.27)
+				)
+				(justify left bottom)
+			)
+		)
+		(property "Manufacturer_Name" "Texas Instruments"
+			(at -519.66 114.3 0)
+			(hide yes)
+			(show_name no)
+			(do_not_autoplace no)
+			(effects
+				(font
+					(size 1.27 1.27)
+				)
+				(justify left bottom)
+			)
+		)
+		(property "Manufacturer_Part_Number" "TPD1E10B06DPYR"
+			(at -619.66 114.3 0)
+			(hide yes)
+			(show_name no)
+			(do_not_autoplace no)
+			(effects
+				(font
+					(size 1.27 1.27)
+				)
+				(justify left bottom)
+			)
+		)
+		(pin "2"
+		)
+		(pin "1"
+		)
+		(instances
+			(project "smart_supply"
+				(path "/487ef637-7a03-4925-80c1-798e0c6f0bbd/f9380e13-e191-4828-b42d-2cc7f479b711"
+					(reference "D14")
+					(unit 1)
+				)

Commit message: MPN BOOT BUTTON MINOR CHANGES
Parts:
- removed C1, C16, C17, C3, C6: 100n, Capacitor_SMD:C_0805_2012Metric, symbol Device:C
- removed C4: 1u, Capacitor_SMD:C_0805_2012Metric, symbol Device:C
- removed F1: Fuse, SmartSupplyLib:fuse holder, symbol Device:Fuse
- added C52, C54, C57, C58, C59, C60: 100n, Capacitor_SMD:C_0805_2012Metric, symbol Device:C
- added R49: 10k, Resistor_SMD:R_0805_2012Metric, symbol Device:R
- added SW2: SW_Push, Button_Switch_SMD:SW_SPST_Omron_B3FS-100xP, symbol Switch:SW_Push
- C14, C56: MPN (none) -> CL21A106KOQNNNE
- C2: MPN (none) -> CL31A226KAHNNNE
- C55: MPN (none) -> CL21A475KAQNNNE
- D14: MPN (none) -> TPD1E10B06DPYR
- D15: MPN (none) -> SMF5V0A-E3-08
- IC4: MPN (none) -> MIC39100-3.3WS-TR
- J10: MPN (none) -> DM3AT-SF-PEJM5
- R19, R20, R21, R22, R23: MPN C17414 -> 0805W8F1002T5E
- R2: MPN (none) -> 0805W8F0000T5E
- R5: MPN (none) -> 0805W8F1002T5E
- SW1: footprint Button_Switch_SMD:Nidec_Copal_CAS-120A -> Button_Switch_SMD:SW_SPST_Omron_B3FS-100xP; MPN (none) -> B3FS-1000P
- U1: MPN (none) -> ESP32-S3-MINI-1U-N8
- U4: MPN (none) -> HLK-10M05
Connections:
- net +3.3V: now also C54.1, C58.2, C60.2, R49.1
- net +5V: now also C55.1; no longer C55.2
- net CH1_L: now also RV2.1, U4.1 (AC/L), C59.2
- net CH1_N: now also C59.1
- net EN: now also C57.2
- net GND: now also C55.2, C52.2, C54.2, C57.1, C58.1, C60.1, SW2.2; no longer C55.1
- net at R2.1, SW1.2: now also C52.1
- net BOOT: now reaches U1.4 (IO0)
- net BOOT: now also R49.2, SW2.1
- no-connect marks 2 -> 23
