File: mcu.kicad_sch (KiCad schematic)
At the start: 33 parts, among them IC4 MIC39100-3.3WS, J1 USB_C_Receptacle_USB2.0_16P, J10 DM3AT-SF-PEJM5, SW1 SW_Push, SW2 SW_Push, U1 ESP32-S3-MINI-1U, U4 HLK-10M05

Commit message: FINAL SCHEMATIC
Global nets, more ESD safety, complete bom, outlets, other fixes, ERC CLEAN
Parts:
- added D16, D17, D18: LED, LED_SMD:LED_0805_2012Metric, symbol Device:LED
- added D6: SS34, Diode_SMD:D_SMA, symbol Diode:SS34
- added H5, H6, H7, H8: MountingHole, MountingHole:MountingHole_3.2mm_M3, symbol Mechanical:MountingHole
- added J16: Conn_01x06_Pin, Connector_JST:JST_XH_B6B-XH-A_1x06_P2.50mm_Vertical, symbol Connector:Conn_01x06_Pin
- added R54, R55, R56: 470, Resistor_SMD:R_0805_2012Metric, symbol Device:R
- added TP1, TP2, TP3: TestPoint, TestPoint:TestPoint_Loop_D2.50mm_Drill1.0mm, symbol Connector:TestPoint
- added U6: USBLC6-2SC6, Package_TO_SOT_SMD:SOT-23-6, symbol Power_Protection:USBLC6-2SC6
- C5: MPN (none) -> ESL227M035AG8AA
- FB1: footprint SmartSupplyLib:fuse holder -> Capacitor_SMD:C_0805_2012Metric; MPN (none) -> BLM21PG221SN1D
- R35: MPN (none) -> 0805W8F1501T5E; now not fitted
- R6, R7: MPN (none) -> 0805W8F5101T5E
Connections:
- net +3.3V: now also TP2.1
- net +5V: now also D6.1 (K), TP1.1; no longer FB1.2
- net GND: now also D16.1 (K), D17.1 (K), D18.1 (K), J16.6 (Pin_6), TP3.1, U6.2 (GND)
- net USB_D+: now also U6.4 (I/O2); no longer J1.A6 (D+), J1.B6 (D+), R35.2
- net USB_D-: now also U6.6 (I/O1); no longer J1.A7 (D-), J1.B7 (D-)
- net LEDSD: now reaches U1.10 (IO6)
- net LEDSD: now also R56.1
- net LED1: now reaches U1.11 (IO7)
- net LED1: now also J16.3 (Pin_3)
- net LED2: now reaches U1.12 (IO8)
- net LED2: now also J16.2 (Pin_2)
- net LED3: now reaches U1.13 (IO9)
- net LED3: now also J16.1 (Pin_1)
- net LEDW: now reaches U1.8 (IO4)
- net LEDW: now also R54.1
- net LEDF: now reaches U1.9 (IO5)
- net LEDF: now also R55.1
- net at FB1.1, J1.A4 (VBUS), J1.A9 (VBUS)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: now also U6.5 (VBUS)
- new net: D18.2 (A), R56.2
- new net: J1.A7 (D-), J1.B7 (D-), U6.1 (I/O1)
- new net: J1.A6 (D+), J1.B6 (D+), R35.2, U6.3 (I/O2)
- new net: D17.2 (A), R55.2
- new net: D6.2 (A), FB1.2
- new net: D16.2 (A), R54.2
- no-connect marks 23 -> 19
Other:
- note added: "AC/DC"
- note added: "BOARD INDICATORS"
- note added: "BOOT"
- note added: "LED JST CONNECTOR"
- note added: "TEST POINTS"
- moved on the sheet: C14, C60, FB1, J10, R19, R20, R21, R22, R23

Commit message: created board
Parts:
- U6: MPN (none) -> USBLC6-2SC6
Changed lines of the file:
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@@
+			)
+		)
+		(property "MPN" "USBLC6-2SC6 "
+			(at 101.6 49.53 0)
+			(hide yes)
+			(show_name no)
+			(do_not_autoplace no)
+			(effects
+				(font
+					(size 1.27 1.27)
+				)
 			)
 		)
